File: CAPSTONE_MC/CAPSTONE_MC.kicad_sch (KiCad schematic)
At the start: 1 part, among them U1 STM32F405RGTx

Commit message: update
Parts:
- added C1, C2, C21, C3, C38, C39, C4, C40, C41, C5, C7, C8, C9: 2.2uF, symbol Device:C
- added C10, C11: 10pF, symbol Device:C
- added C12: 100nF, symbol Device:C
- added C13: 2.2uF 450V, symbol Device:C_Polarized
- added C14: 2.2uF 50V, symbol Device:C
- added C15: 100nF 25V, symbol Device:C
- added C16: 100uF 25V, symbol Device:C
- added C17: 100nF 450V, symbol Device:C
- added C18, C19: 10uF, symbol Device:C
- added C20: 100nF 16V, symbol Device:C
- added C22: 47pF DNF, symbol Device:C
- added C23, C24, C25, C29, C30, C31, C32, C33, C42, C6: C, symbol Device:C
- added C26, C27, C28: 1uF, symbol Device:C
- added C34: C_Polarized, symbol Device:C_Polarized
- added C35, C36, C37: 4.7nF, symbol Device:C
- added C43, C44: 33pF, symbol Device:C
- added D1, D3: SURS8360BT3G, symbol Device:D
- added D10, D8, D9: D_Schottky, symbol Device:D_Schottky
- added D11: D_TVS_Dual_AAC, symbol Device:D_TVS_Dual_AAC
- added D2: 10V BZT52C10, symbol Device:D_Zener
- added D4: PMEG6020ER, symbol Device:D_Schottky
- added D5: BLUE, symbol Device:LED
- added D6: RED, symbol Device:LED
- added D7: GREEN, symbol Device:LED
- added J1: USB_C_Receptacle_USB2.0_16P, symbol Connector:USB_C_Receptacle_USB2.0_16P
- added J2: Conn_01x03, symbol Connector_Generic:Conn_01x03
- added J3: Conn_01x02, symbol Connector_Generic:Conn_01x02
- added L1: L, symbol Device:L
- added L2: 1mH >600mA, symbol Device:L
- added L3: 10uH >1.2A <200mR, symbol Device:L
- added NT1: NetTie_2, symbol Device:NetTie_2
- added R1: 1R 1206, symbol Device:R
- added R10, R11, R12: R_Shunt, symbol Device:R_Shunt
- added R13, R14, R15: 100R, symbol Device:R
- added R16, R17: 10K, symbol Device:R
- added R18, R19: 5K1, symbol Device:R
- added R2: 13K, symbol Device:R
- added R20: 120R, symbol Device:R
- added R21: 0R, symbol Device:R
- added R3: 4K3, symbol Device:R
- added R4, R5, R6: 1K, symbol Device:R
- added R7, R8, R9: R, symbol Device:R
- added SW1, SW2: SW_Push, symbol Switch:SW_Push
- added TH1: 10K_NTC, symbol Device:Thermistor_NTC
- added TH2: 10K_NTC or CNT, symbol Device:Thermistor_NTC
- added U10: ~, symbol RLX_Library:EG1120
- added U11: LGS5145, Package_TO_SOT_SMD:SOT-23-6, symbol Regulator_Switching:LGS5145
- added U2, U3, U4: LAS1M0750, RLX_Library:LasSOP-10, symbol RLX_Library:LAS1M0750
- added U5, U6, U7: INA181, Package_TO_SOT_SMD:SOT-23-6, symbol Amplifier_Current:INA181
- added U8: AS5047D, Package_SO:TSSOP-14_4.4x5mm_P0.65mm, symbol Sensor_Magnetic:AS5047D
- added U9: SN65HVD232, Package_SO:SOIC-8_3.9x4.9mm_P1.27mm, symbol Interface_CAN_LIN:SN65HVD232
- added Y1: Crystal_GND24, symbol Device:Crystal_GND24
Connections:
- net +3V3: now reaches U1.1 (VBAT)
- net +3V3: now also U1.19 (VDD), U1.32 (VDD), U1.48 (VDD), U1.64 (VDD), C1.1, C19.1, C2.1, C22.1, C3.1, C4.1, C42.1, L1.2, L3.2, R2.1, R6.1, U9.3 (VCC)
- net CURRENT_3: now reaches U1.10 (PC2)
- net CURRENT_3: now also C35.1, R13.1
- net AN_IN: now reaches U1.11 (PC3)
- net GNDA: now reaches U1.12 (VSSA)
- net GNDA: now also C21.2, C35.2, C36.2, C37.2, C38.2, C39.2, C40.2, C41.2, C5.2, C6.1, C7.2, NT1.2, R16.2, R17.2, U5.2 (GND), U6.2 (GND), U7.2 (GND)
- net +3.3VA: now reaches U1.13 (VDDA)
- net +3.3VA: now also C21.1, C38.1, C39.1, C5.1, C6.2, C7.1, L1.1, TH1.1, TH2.1, U5.6 (V+), U6.6 (V+), U7.6 (V+)
- net VOLTAGE_1: now reaches U1.14 (PA0)
- net VOLTAGE_2: now reaches U1.15 (PA1)
- net VOLTAGE_3: now reaches U1.16 (PA2)
- net ADC_TEMP: now reaches U1.17 (PA3)
- net ADC_TEMP: now also C40.1, R16.1, TH1.2
- net GND: now reaches U1.18 (VSS), U1.63 (VSS)
- net GND: now also U1.60 (BOOT0), C1.2, C10.2, C11.2, C12.2, C13.2, C15.2, C16.2, C17.2, C18.2, C19.2, C2.2, C26.2, C27.2, C28.2, C3.2, C4.2, C42.2, C43.2, C44.1, C8.2, C9.2, D1.2 (A), D11.3 (common), D4.2 (A), D5.1 (K), D6.1 (K), D7.1 (K), J1.A1 (GND), J1.A12 (GND), J1.B1 (GND), J1.B12 (GND), J1.S1 (SHIELD), J3.2 (Pin_2), NT1.1, R10.4, R11.4, R12.4, R18.2, R19.2, R3.1, SW1.2, SW2.2, U11.2 (GND), U2.10 (GND), U3.10 (GND), U4.10 (GND), U9.2 (GND), Y1.2, Y1.4
- net RX_SDA_NSS: now reaches U1.20 (PA4)
- net RX_SDA_NSS: now also U1.30 (PB11), U8.1 (~{CS})
- net SCK_ADC_EXT: now reaches U1.21 (PA5)
- net SCK_ADC_EXT: now also U8.2 (CLK)
- net MISO_ADC_EXT2: now reaches U1.22 (PA6)
- net MISO_ADC_EXT2: now also U8.3 (MISO)
- net TX_SCL_MOSI: now reaches U1.23 (PA7)
- net TX_SCL_MOSI: now also U1.29 (PB10), U8.4 (MOSI)
- net TEMP_MOTOR: now reaches U1.24 (PC4)
- net TEMP_MOTOR: now also C41.1, R17.1, TH2.2
- net ADC_15: now reaches U1.25 (PC5)
- net LED_BLUE: now reaches U1.26 (PB0)
- net LED_BLUE: now also R4.1
- net LED_RED: now reaches U1.27 (PB1)
- net LED_RED: now also R5.1
- net at U1.31 (VCAP_1): now also C9.1
- net PB12: now reaches U1.33 (PB12)
- net L1: now reaches U1.34 (PB13)
- net L1: now also U2.7 (INL)
- net L2: now reaches U1.35 (PB14)
- net L2: now also U3.7 (INL)
- net L3: now reaches U1.36 (PB15)
- net L3: now also U4.7 (INL)
- net HALL_1: now reaches U1.37 (PC6)
- net HALL_2: now reaches U1.38 (PC7)
- net HALL_3: now reaches U1.39 (PC8)
- net SPI3_CS: now reaches U1.40 (PC9)
- net H1: now reaches U1.41 (PA8)
- net H1: now also U2.6 (INH)
- net H2: now reaches U1.42 (PA9)
- net H2: now also U3.6 (INH)
- net H3: now reaches U1.43 (PA10)
- net H3: now also U4.6 (INH)
- net USB_DM: now reaches U1.44 (PA11)
- net USB_DM: now also J1.A7 (D-), J1.B7 (D-)
- net USB_DP: now reaches U1.45 (PA12)
- net USB_DP: now also J1.A6 (D+), J1.B6 (D+)
- net SWDIO: now reaches U1.46 (PA13)
- net at U1.47 (VCAP_2): now also C8.1
- net SWCLK: now reaches U1.49 (PA14)
- net OSC_IN: now reaches U1.5 (PH0)
- net OSC_IN: now also C10.1, Y1.1
- net SPI3_SCK: now reaches U1.51 (PC10)
- net SPI3_MISO: now reaches U1.52 (PC11)
- net SPI3_MOSI: now reaches U1.53 (PC12)
- net PD2: now reaches U1.54 (PD2)
- net PB3: now reaches U1.55 (PB3)
- net PB4: now reaches U1.56 (PB4)
- net EN_GATE: now reaches U1.57 (PB5)
- net U1_TX_SERVO: now reaches U1.58 (PB6)
- net U1_RX_FAULT: now reaches U1.59 (PB7)
- net OSC_OUT: now reaches U1.6 (PH1)
- net OSC_OUT: now also C11.1, Y1.3
- net CAN_RX: now reaches U1.61 (PB8)
- net CAN_RX: now also U9.4 (R)
- net CAN_TX: now reaches U1.62 (PB9)
- net CAN_TX: now also U9.1 (D)
- net nRST: now reaches U1.7 (NRST)
- net nRST: now also C12.1, SW1.1
- net CURRENT_1: now reaches U1.8 (PC0)
- net CURRENT_1: now also C37.1, R15.1
- net CURRENT_2: now reaches U1.9 (PC1)
- net CURRENT_2: now also C36.1, R14.1
- new net: C28.1, R8.2, U4.5 (VCC)
- new net: D7.2 (A), R6.2
- new net: R1.1, U10.3 (CS)
- new net: C14.1, D1.1 (K), L2.1, R1.2
- new net: R10.2, U5.3 (+)
- new net: R10.3, U5.4 (-)
- new net: D2.1 (K), D3.1 (K)
- new net: C20.1, U11.1 (BST)
- new net: C22.2, R2.2, R3.2, U11.3 (FB)
- new net: C20.2, D4.1 (K), L3.1, U11.6 (SW)
- new net: D10.2 (A), R9.1
- new net: C26.1, R9.2, U2.5 (VCC)
- new net: C24.1, D9.1 (K), U4.4 (BST)
- new net: D9.2 (A), R8.1
- new net: C14.2, D2.2 (A), U10.2 (VDD)
- new net: C23.1, D8.1 (K), U3.4 (BST)
- new net: C23.2, J2.2 (Pin_2), U3.2 (SW)
- new net: C24.2, J2.3 (Pin_3), U4.2 (SW)
- new net: R10.1, U4.1 (VS)
- new net: C25.1, D10.1 (K), U2.4 (BST)
- new net: C25.2, J2.1 (Pin_1), U2.2 (SW)
- new net: R12.1, U2.1 (VS)
- new net: R11.2, U6.3 (+)
- new net: R11.3, U6.4 (-)
- new net: R20.2, R21.1
- new net: D8.2 (A), R7.1
- new net: C27.1, R7.2, U3.5 (VCC)
- new net: R12.2, U7.3 (+)
- new net: R12.3, U7.4 (-)
- new net: J1.A4 (VBUS), J1.A9 (VBUS), J1.B4 (VBUS), J1.B9 (VBUS)
- new net: J1.A5 (CC1), R18.1
- new net: J1.B5 (CC2), R19.1
- new net: R11.1, U3.1 (VS)
- new net: D6.2 (A), R5.2
- new net: D5.2 (A), R4.2
- new net +15V: C15.1, C16.1, C18.1, D3.2 (A), L2.2, U11.4 (EN), U11.5 (VIN)
- new net CANH: C43.1, D11.1 (A1), R20.1, U9.7 (CANH)
- new net CANL: C44.2, D11.2 (A2), R21.2, U9.6 (CANL)
- new net C_A: R15.2, U7.1
- new net C_B: R14.2, U6.1
- new net C_C: R13.2, U5.1
- new net HVBUS: C13.1, C17.1, J3.1 (Pin_1), U10.1 (Drain), U2.3 (VIN), U3.3 (VIN), U4.3 (VIN)
- no-connect marks 0 -> 8
Other:
- moved on the sheet: U1

Commit message: 1. 更新PCB v1.0.0 2. 更新规格书
Parts:
- removed C13: 2.2uF 450V, symbol Device:C_Polarized
- removed C34: C_Polarized, symbol Device:C_Polarized
- removed J1: USB_C_Receptacle_USB2.0_16P, symbol Connector:USB_C_Receptacle_USB2.0_16P
- removed J2: Conn_01x03, symbol Connector_Generic:Conn_01x03
- removed J3: Conn_01x02, symbol Connector_Generic:Conn_01x02
- removed R10, R11, R12: R_Shunt, symbol Device:R_Shunt
- removed R18, R19: 5K1, symbol Device:R
- removed SW1, SW2: SW_Push, symbol Switch:SW_Push
- added C13, C45: 100nF, Capacitor_SMD:C_0402_1005Metric, symbol Device:C
- added C34: 22uF, Capacitor_SMD:C_0805_2012Metric, symbol Device:C
- added C46, C47: 1uF, Capacitor_SMD:C_0402_1005Metric, symbol Device:C
- added C48, C49, C50: 2.2uF 450V, Capacitor_SMD:C_2220_5750Metric, symbol Device:C
- added C51: 10uF, Capacitor_SMD:C_0402_1005Metric, symbol Device:C
- added C54, C55: 2.2uF, Capacitor_SMD:C_0402_1005Metric, symbol Device:C
- added H1, H2, H3: MountingHole, MountingHole:MountingHole_2.2mm_M2, symbol Mechanical:MountingHole
- added R10, R11, R12: 7mR, Resistor_SMD:R_1206_3216Metric, symbol Device:R
- added R22, R24, R26, R28: 137K, Resistor_SMD:R_1206_3216Metric, symbol Device:R
- added R23, R25, R27, R29: 1K, Resistor_SMD:R_0402_1005Metric, symbol Device:R
- added R30, R31: 3K3, Resistor_SMD:R_0402_1005Metric, symbol Device:R
- added R32, R33: 22R, Resistor_SMD:R_0402_1005Metric, symbol Device:R
- added SYM1: Logo_Open_Hardware_Small, RLX_Library:OSHW-Logo_5.7x6mm_SilkScreen_noText, symbol Graphic:Logo_Open_Hardware_Small
- added SYM3: SYM_Flash_Large, Symbol:Symbol_HighVoltage_NoTriangle_2x5mm_Copper, symbol Graphic:SYM_Flash_Large
- added SYM5: Logo_Open_Hardware_Small, Symbol:KiCad-Logo_5mm_SilkScreen, symbol Graphic:Logo_Open_Hardware_Small
- added TP1, TP17, TP18, TP19, TP2, TP3, TP4, TP5: TestPoint, TestPoint:TestPoint_Pad_D1.5mm, symbol Connector:TestPoint
- added TP10, TP11, TP12, TP13, TP14, TP15, TP16, TP20, TP21, TP6, TP7, TP8, TP9: TestPoint, TestPoint:TestPoint_Pad_D1.0mm, symbol Connector:TestPoint
- added U12: XC6220B331MR, Package_TO_SOT_SMD:SOT-23-5, symbol Regulator_Linear:XC6220B331MR
- added U13: LMV321, Package_TO_SOT_SMD:SOT-23-5, symbol Amplifier_Operational:LMV321
- C1, C10, C11, C12, C19, C2, C21, C3, C38, C39, C4, C40, C41, C43, C44, C5, C7, C8, C9: footprint (none) -> Capacitor_SMD:C_0402_1005Metric
- C14, C18, C26, C27, C28: footprint (none) -> Capacitor_SMD:C_0603_1608Metric
- C15: value 100nF 25V -> 100nF; footprint (none) -> Capacitor_SMD:C_0402_1005Metric
- C16: value 100uF 25V -> 22uF; footprint (none) -> Capacitor_SMD:C_0805_2012Metric
- C17: footprint (none) -> Capacitor_SMD:C_1206_3216Metric
- C20: value 100nF 16V -> 100nF; footprint (none) -> Capacitor_SMD:C_0402_1005Metric
- C22: value 47pF DNF -> 47pF DNP; footprint (none) -> Capacitor_SMD:C_0402_1005Metric; now not fitted
- C23, C24, C25: value C -> 220nF; footprint (none) -> Capacitor_SMD:C_0402_1005Metric
- C29, C33: value C -> 10uF; footprint (none) -> Capacitor_SMD:C_0402_1005Metric
- C30, C31, C32: value C -> 2.2uF 450V; footprint (none) -> Capacitor_SMD:C_2220_5750Metric
- C35, C36, C37: footprint (none) -> Capacitor_SMD:C_0402_1005Metric; now not fitted
- C42: value C -> 100nF; footprint (none) -> Capacitor_SMD:C_0402_1005Metric
- C6: value C -> 1uF; footprint (none) -> Capacitor_SMD:C_0402_1005Metric
- D1, D3: footprint (none) -> Diode_SMD:D_SMB
- D10, D8, D9: value D_Schottky -> US1JW; footprint (none) -> Diode_SMD:D_SOD-123F
- D11: value D_TVS_Dual_AAC -> PESD1CAN; footprint (none) -> Package_TO_SOT_SMD:SOT-23
- D2: footprint (none) -> Diode_SMD:D_SOD-123
- D4: value PMEG6020ER -> SS24L; footprint (none) -> Diode_SMD:D_SOD-123F
- D5, D6, D7: footprint (none) -> LED_SMD:LED_0402_1005Metric
- L1: value L -> 0R; footprint (none) -> Inductor_SMD:L_0402_1005Metric
- L2: footprint (none) -> Inductor_SMD:L_Bourns_SRN8040TA
- L3: footprint (none) -> Inductor_SMD:L_Abracon_ASPI-0425
- NT1: footprint (none) -> NetTie:NetTie-2_SMD_Pad0.5mm
- R1: value 1R 1206 -> 1R; footprint (none) -> Resistor_SMD:R_1206_3216Metric
- R13, R14, R15, R16, R17, R2, R20, R21, R4, R5, R6, TH1, TH2: footprint (none) -> Resistor_SMD:R_0402_1005Metric
- R3: value 4K3 -> 3K4; footprint (none) -> Resistor_SMD:R_0402_1005Metric
- R7, R8, R9: value R -> 10R; footprint (none) -> Resistor_SMD:R_0805_2012Metric
- U10: value ~ -> EG1120; footprint (none) -> Package_TO_SOT_SMD:SOT-23-3
- U5, U6, U7: value INA181 -> INA181A1
- Y1: footprint (none) -> Crystal:Crystal_SMD_3225-4Pin_3.2x2.5mm
Connections:
- net +15V: now also C26.1, C27.1, C28.1, R7.2, R8.2, R9.2, U2.5 (VCC), U3.5 (VCC), U4.5 (VCC), C34.1
- net +3.3VA: now also C47.1, R30.1, U13.5 (V+)
- net +3V3: now also C33.1, R4.1, U8.11 (VDD), U8.12 (VDD3V3), C13.1, C45.1, C51.1, C54.1, C55.1, TP21.1, U12.5 (VOUT); no longer C19.1, C22.1, L3.2, R2.1, R6.1
- net AN_IN: now also R22.1, R23.1
- net CANH: now also TP13.1, TP15.1
- net CANL: now also TP14.1, TP16.1
- net GND: now also C29.2, C30.2, C31.2, C32.2, C33.2, U5.4 (-), U6.4 (-), U7.4 (-), U8.13 (GND), U8.5 (TST), C13.2, C34.2, C45.2, C48.2, C49.2, C50.2, C51.2, C54.2, C55.2, R10.2, R11.2, R12.2, R23.2, R25.2, R27.2, R29.2, TP12.1, TP2.1, TP20.1, U12.2 (GND)
- net GNDA: now also C46.2, C47.2, R31.2, U13.2 (V-)
- net HVBUS: now also C30.1, C31.1, C32.1, C48.1, C49.1, C50.1, R22.2, TP1.1
- net RX_SDA_NSS: no longer U1.30 (PB11)
- net SWCLK: now also TP11.1
- net SWDIO: now also TP10.1
- net TX_SCL_MOSI: no longer U1.29 (PB10)
- net U1_RX_FAULT: now also TP8.1
- net U1_TX_SERVO: now also TP9.1
- net USB_DM: now also R32.2
- net USB_DP: now also R33.2
- net VOLTAGE_1: now also R24.1, R25.1
- net VOLTAGE_2: now also R26.1, R27.1
- net VOLTAGE_3: now also R28.1, R29.1
- net at U5.3 (+): now also U4.1 (VS), R10.1
- net Vref: now reaches U5.5 (REF)
- net Vref: now also U6.5 (REF), U7.5 (REF), U13.3 (-), U13.4
- net HS2: now reaches C23.2, U3.2 (SW)
- net HS2: now also R26.2, TP18.1, TP4.1
- net HS3: now reaches C24.2, U4.2 (SW)
- net HS3: now also R28.2, TP19.1, TP5.1
- net BTN: now reaches U1.2 (PC13)
- net HS1: now reaches C25.2, U2.2 (SW)
- net HS1: now also R24.2, TP17.1, TP3.1
- net at U2.1 (VS): now also U7.3 (+), R12.1
- net at U6.3 (+): now also U3.1 (VS), R11.1
- net +3V8: now reaches C29.1
- net +3V8: now also C19.1, C22.1, L3.2, R2.1, U12.1 (VIN), U12.3 (CE)
- net EN_GATE: no longer names the net of U1.57 (PB5)
- net LED_BLUE renamed LED_GREEN
- net LED_GREEN: now also R6.1; no longer R4.1
- net PB12: no longer names the net of U1.33 (PB12)
- net PB3: no longer names the net of U1.55 (PB3)
- net PB4: no longer names the net of U1.56 (PB4)
- net PD2: no longer names the net of U1.54 (PD2)
- new net: R32.1, TP6.1
- new net: C46.1, R30.2, R31.1, U13.1 (+)
- new net: R33.1, TP7.1
- no-connect marks 8 -> 25
Other:
- note added: "修正为3.9167V"
- moved on the sheet: C1, C10, C11, C12, C18, C19, C2, C20, C21, C23, C24, C25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
